File: RobotFish.brd (EAGLE design)
At the start: 160 x 100 mm, 14 parts, among them U1 MCP73831/OT, U3 MCP1754S_SOT23

Commit message: schematics
Parts:
- added C1, C2, C7: 0.1uF, water:C0603(1608)
- added C5: 10nF, water:C0603(1608)
- added C6: (no value), water:C0805(2012)
- added R10, R5, R6: 100k, water:R0603(1608)
- added R7, R8, R9: (no value), water:R0603(1608)
- added TR1: SSM3J338R, water:SOT23
- added U2: 16F1575, water:SO-14
- added U4: LMC555, water:SO8
Connections:
- net N$5 renamed VIN
- removed net PGEC: JP2.5
- removed net PGED: JP2.4
- new net ADC: R3.1, R4.2, U2.10
- new net ICSPCLK: JP2.5, U2.12
- new net ICSPDAT: JP2.4, U2.13
- new net N$11: C5.2, U4.5
- new net N$12: R7.1
- new net N$13: R8.2
- new net N$8: TR1.3
- new net N$9: C6.1, R8.1, U4.2, U4.6
- new net RX: U2.5
- new net SERVO_ON: R6.1, TR1.1, U2.9
- new net SERVO_PWM: R9.1
- new net T1CKI: R7.2, U2.2, U4.3
- new net T1G: U2.3
- new net TX: U2.6
- net +3.3V: now also C1.2, C2.1, R10.2, U2.1, U4.8
- net +5V: now also R5.2
- net DGND: now also C1.1, C2.2, C5.1, C6.2, C7.2, R5.1, U2.14, U4.1
- net N$4: now also R9.2, U2.8; no longer R3.1, R4.2
- net RESET: now also C7.1, R10.1, U2.4
- net VBAT: now also R6.2, TR1.2
Changed lines of the file:
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@@
 <element name="R4" library="water" package="R0603(1608)" value="100k" x="-7.62" y="-67.31"/>
 <element name="D1" library="microbuilder" package="SOD-123" value="MBR120" x="-6.35" y="-72.39"/>
+<element name="U2" library="water" package="SO-14" value="16F1575" x="-3.81" y="-81.28"/>
+<element name="R5" library="water" package="R0603(1608)" value="100k" x="-7.62" y="-88.9"/>
+<element name="U4" library="water" package="SO8" value="LMC555" x="-5.08" y="-97.79"/>
+<element name="TR1" library="water" package="SOT23" value="SSM3J338R" x="-7.62" y="-105.41"/>
+<element name="R6" library="water" package="R0603(1608)" value="100k" x="-7.62" y="-111.76"/>
+<element name="C1" library="water" package="C0603(1608)" value="0.1uF" x="-7.62" y="-118.11"/>
+<element name="C2" library="water" package="C0603(1608)" value="0.1uF" x="-7.62" y="-121.92"/>
+<element name="C5" library="water" package="C0603(1608)" value="10nF" x="-7.62" y="-128.27"/>
+<element name="C6" library="water" package="C0805(2012)" value="" x="-7.62" y="-134.62"/>
+<element name="R7" library="water" package="R0603(1608)" value="" x="-7.62" y="-138.43"/>
+<element name="R8" library="water" package="R0603(1608)" value="" x="-7.62" y="-142.24"/>
+<element name="R9" library="water" package="R0603(1608)" value="" x="-7.62" y="-146.05"/>
+<element name="R10" library="water" package="R0603(1608)" value="100k" x="-7.62" y="-149.86"/>
+<element name="C7" library="water" package="C0603(1608)" value="0.1uF" x="-7.62" y="-156.21"/>
 </elements>
 <signals>
@@
 <contactref element="CN1" pad="1"/>
 <contactref element="R4" pad="1"/>
+<contactref element="U2" pad="14"/>
+<contactref element="R5" pad="1"/>
+<contactref element="U4" pad="1"/>
+<contactref element="C1" pad="1"/>
+<contactref element="C5" pad="1"/>
+<contactref element="C6" pad="2"/>
+<contactref element="C2" pad="2"/>
+<contactref element="C7" pad="2"/>
+<wire x1="-6.62" y1="-134.62" x2="-6.87" y2="-156.21" width="0" layer="19" extent="1-1"/>
+<wire x1="-8.37" y1="-128.27" x2="-6.62" y2="-134.62" width="0" layer="19" extent="1-1"/>
+<wire x1="-6.87" y1="-121.92" x2="-8.37" y2="-128.27" width="0" layer="19" extent="1-1"/>
+<wire x1="-8.37" y1="-118.11" x2="-6.87" y2="-121.92" width="0" layer="19" extent="1-1"/>
+<wire x1="-6.985" y1="-100.49" x2="-8.37" y2="-118.11" width="0" layer="19" extent="1-1"/>
+<wire x1="-8.37" y1="-88.9" x2="-6.985" y2="-100.49" width="0" layer="19" extent="1-1"/>
+<wire x1="-7.62" y1="-78.68" x2="-8.37" y2="-88.9" width="0" layer="19" extent="1-1"/>
+<wire x1="-8.37" y1="-67.31" x2="-7.62" y2="-78.68" width="0" layer="19" extent="1-1"/>
 <wire x1="-5.83" y1="-48.26" x2="-8.37" y2="-67.31" width="0" layer="19" extent="1-1"/>
 <wire x1="-1.24" y1="-38.1" x2="-5.83" y2="-48.26" width="0" layer="19" extent="1-1"/>
@@
 <contactref element="U3" pad="2"/>
 <contactref element="C4" pad="1"/>
+<contactref element="U2" pad="1"/>
+<contactref element="C1" pad="2"/>
+<contactref element="U4" pad="8"/>
+<contactref element="C2" pad="1"/>
+<contactref element="R10" pad="2"/>
+<wire x1="-8.37" y1="-121.92" x2="-6.87" y2="-149.86" width="0" layer="19" extent="1-1"/>
+<wire x1="-6.87" y1="-118.11" x2="-8.37" y2="-121.92" width="0" layer="19" extent="1-1"/>
+<wire x1="-6.985" y1="-95.09" x2="-6.87" y2="-118.11" width="0" layer="19" extent="1-1"/>
+<wire x1="-7.62" y1="-83.88" x2="-6.985" y2="-95.09" width="0" layer="19" extent="1-1"/>
+<wire x1="-3.84" y1="-38.1" x2="-7.62" y2="-83.88" width="0" layer="19" extent="1-1"/>
 <wire x1="-2.86" y1="-25.23" x2="-3.84" y2="-38.1" width="0" layer="19" extent="1-1"/>
 <wire x1="5.08" y1="-3.81" x2="-2.86" y2="-25.23" width="0" layer="19" extent="1-1"/>
@@
 <signal name="RESET">
 <contactref element="JP2" pad="1"/>
+<contactref element="U2" pad="4"/>
+<contactref element="R10" pad="1"/>
+<contactref element="C7" pad="1"/>
+<wire x1="-8.37" y1="-149.86" x2="-8.37" y2="-156.21" width="0" layer="19" extent="1-1"/>
+<wire x1="-3.81" y1="-83.88" x2="-8.37" y2="-149.86" width="0" layer="19" extent="1-1"/>
+<wire x1="2.54" y1="-3.81" x2="-3.81" y2="-83.88" width="0" layer="19" extent="1-1"/>
 </signal>
-<signal name="PGED">
+<signal name="ICSPDAT">
 <contactref element="JP2" pad="4"/>
+<contactref element="U2" pad="13"/>
+<wire x1="10.16" y1="-3.81" x2="-6.35" y2="-78.68" width="0" layer="19" extent="1-1"/>
 </signal>
-<signal name="PGEC">
+<signal name="ICSPCLK">
 <contactref element="JP2" pad="5"/>
+<contactref element="U2" pad="12"/>
+<wire x1="12.7" y1="-3.81" x2="-5.08" y2="-78.68" width="0" layer="19" extent="1-1"/>
 </signal>
 <signal name="VBAT">
@@
 <contactref element="R3" pad="2"/>
 <contactref element="U1" pad="3"/>
+<contactref element="TR1" pad="2"/>
+<contactref element="R6" pad="2"/>
+<wire x1="-6.67" y1="-106.51" x2="-6.87" y2="-111.76" width="0" layer="19" extent="1-1"/>
+<wire x1="-6.87" y1="-60.96" x2="-6.67" y2="-106.51" width="0" layer="19" extent="1-1"/>
 <wire x1="-1.96" y1="-43.18" x2="-6.87" y2="-60.96" width="0" layer="19" extent="1-1"/>
 <wire x1="3.49" y1="-10.19" x2="-1.96" y2="-43.18" width="0" layer="19" extent="1-1"/>
@@
 <contactref element="LED1" pad="A"/>
 <contactref element="D1" pad="A"/>
+<contactref element="R5" pad="2"/>
+<wire x1="-4.5" y1="-72.39" x2="-6.87" y2="-88.9" width="0" layer="19" extent="1-1"/>
 <wire x1="-8.89" y1="-49.01" x2="-4.5" y2="-72.39" width="0" layer="19" extent="1-1"/>
 <wire x1="-2.685" y1="-31.75" x2="-8.89" y2="-49.01" width="0" layer="19" extent="1-1"/>
@@
 <wire x1="-8.89" y1="-47.51" x2="-8.37" y2="-54.61" width="0" layer="19" extent="1-1"/>
 </signal>
-<signal name="N$4">
+<signal name="ADC">
 <contactref element="R4" pad="2"/>
 <contactref element="R3" pad="1"/>
+<contactref element="U2" pad="10"/>
+<wire x1="-6.87" y1="-67.31" x2="-2.54" y2="-78.68" width="0" layer="19" extent="1-1"/>
 <wire x1="-8.37" y1="-60.96" x2="-6.87" y2="-67.31" width="0" layer="19" extent="1-1"/>
 </signal>
-<signal name="N$5">
+<signal name="VIN">
 <contactref element="U3" pad="3"/>
 <contactref element="C3" pad="1"/>
@@
 <wire x1="-3.81" y1="-23.03" x2="2.51" y2="-31.75" width="0" layer="19" extent="1-1"/>
 </signal>
+<signal name="N$8">
+<contactref element="TR1" pad="3"/>
+</signal>
+<signal name="N$11">
+<contactref element="U4" pad="5"/>
+<contactref element="C5" pad="2"/>
+<wire x1="-3.175" y1="-95.09" x2="-6.87" y2="-128.27" width="0" layer="19" extent="1-1"/>
+</signal>
+<signal name="N$9">
+<contactref element="U4" pad="2"/>
+<contactref element="U4" pad="6"/>
+<contactref element="C6" pad="1"/>
+<contactref element="R8" pad="1"/>
+<wire x1="-8.62" y1="-134.62" x2="-8.37" y2="-142.24" width="0" layer="19" extent="1-1"/>
+<wire x1="-5.715" y1="-100.49" x2="-8.62" y2="-134.62" width="0" layer="19" extent="1-1"/>
+<wire x1="-4.445" y1="-95.09" x2="-5.715" y2="-100.49" width="0" layer="19" extent="1-1"/>
+</signal>
+<signal name="N$12">
+<contactref element="R7" pad="1"/>
+</signal>
+<signal name="N$13">
+<contactref element="R8" pad="2"/>
+</signal>
+<signal name="T1CKI">
+<contactref element="U2" pad="2"/>
+<contactref element="U4" pad="3"/>
+<contactref element="R7" pad="2"/>
+<wire x1="-4.445" y1="-100.49" x2="-6.87" y2="-138.43" width="0" layer="19" extent="1-1"/>
+<wire x1="-6.35" y1="-83.88" x2="-4.445" y2="-100.49" width="0" layer="19" extent="1-1"/>
+</signal>
+<signal name="T1G">
+<contactref element="U2" pad="3"/>
+</signal>
+<signal name="SERVO_ON">
+<contactref element="R6" pad="1"/>
+<contactref element="TR1" pad="1"/>
+<contactref element="U2" pad="9"/>
+<wire x1="-8.57" y1="-106.51" x2="-8.37" y2="-111.76" width="0" layer="19" extent="1-1"/>
+<wire x1="-1.27" y1="-78.68" x2="-8.57" y2="-106.51" width="0" layer="19" extent="1-1"/>
+</signal>
+<signal name="RX">
+<contactref element="U2" pad="5"/>
+</signal>
+<signal name="TX">
+<contactref element="U2" pad="6"/>
+</signal>
+<signal name="N$4">
+<contactref element="U2" pad="8"/>
+<contactref element="R9" pad="2"/>
+<wire x1="0" y1="-78.68" x2="-6.87" y2="-146.05" width="0" layer="19" extent="1-1"/>
+</signal>
+<signal name="SERVO_PWM">
+<contactref element="R9" pad="1"/>
+</signal>
 </signals>

Commit message: almost done
Parts:
- removed C5: 10nF, water:C0603(1608)
- removed C6: (no value), water:C0805(2012)
- removed C7: 0.1uF, water:C0603(1608)
- removed D4: MBR120, microbuilder:SOD-123
- removed JP2: (no value), SparkFun-Connectors:1X05
- removed TVS2: SD05C, berry:SOD-323-NOPOL
- removed U4: LMC555, water:SO8
- added D2, D3: MBR120, microbuilder:SOD-123
- added JP1: (no value), SparkFun-Connectors:1X05
- added LED2: (no value), berry:LED-0603
- added LED3: (no value), berry:LED3MM
- added R11, R13: 10k, water:R0603(1608)
- added R12: 1k, water:R0603(1608)
- added R14: 100k, water:R0603(1608)
- added TP1, TP2, TP3, TP4: (no value), water:TP-5010
- added TVS1: SD05C, berry:SOD-323-NOPOL
- added X1: JST_3PIN, water:SM03B-SRSS-TB
- CN1: device adafruit:JST-PH-2-THM-RA -> water:JST-PH-2-THM-RA
- R1: value 10k -> 100k
- R10, R3, R4: value 100k -> (none)
- R2: value 1k -> 100k
- R5: value 100k -> 10k
- R6: value 100k -> 1k
- R7: value (none) -> 1k
- R8, R9: value (none) -> 100k
- U1: value MCP73831/OT -> 16F1575; device water:SOT23-5L -> water:SO-14
- U2: value 16F1575 -> MCP73831/OT; device water:SO-14 -> water:SOT23-5L
- moved R7 167.1 mm to (25.4, 25.4), turned to 90 degrees
- moved R9 166.1 mm to (26.7, 16.5)
- moved R8 163.0 mm to (29.2, 16.5)
- moved R10 159.2 mm to (22.9, 6.35)
- moved C2 141.6 mm to (15.2, 17.8)
- moved C1 131.6 mm to (6.35, 12.7), turned to 270 degrees
- moved TR1 131.3 mm to (47.0, 14.0), turned to 270 degrees
- moved R5 117.4 mm to (19.1, 25.4)
- moved R6 116.1 mm to (3.81, 3.81), turned to 180 degrees
- moved U2 112.4 mm to (22.9, 27.9), turned to 90 degrees
- moved D1 102.9 mm to (10.2, 29.2), turned to 180 degrees
- moved R2 82.5 mm to (12.7, 25.4), turned to 90 degrees
- moved C4 82.3 mm to (48.3, 26.7), turned to 270 degrees
- moved R4 76.5 mm to (7.62, 7.62), turned to 180 degrees
- moved U3 74.8 mm to (44.5, 33.0), turned to 90 degrees
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Connections:
- removed net ADC: R3.1, R4.2, U2.10
- removed net N$11: C5.2, U4.5
- removed net N$12: R7.1
- removed net N$13: R8.2
- removed net N$9: C6.1, R8.1, U4.2, U4.6
- removed net T1CKI: R7.2, U2.2, U4.3
- removed net T1G: U2.3
- new net BAT_ADC: R8.1, R9.2, U1.3
- new net LED_STAT: R6.1, U1.7
- new net N$15: R11.2, TP3.TP
- new net N$16: R12.2, TP4.TP
- new net N$5: D1.A, TP1.TP
- new net N$6: R3.1, U1.5
- new net N$7: R4.1, U1.6
- new net SERVO_POWER: TR1.3, X1.2
- new net W_IN: R12.1, R13.2, U1.10
- new net W_OUT: R11.1, U1.11
- net +3.3V: now also JP1.2, R1.2, U1.1; no longer C1.2, JP2.2, R10.2, U2.1, U4.8
- net +5V: now also D1.C, D2.A, LED2.A, R2.2, TVS1.2, U2.4; no longer D1.A, LED1.A, R5.2, TVS2.2, U1.4
- net DGND: now also C1.2, CN1.2, JP1.3, LED1.C, LED3.K, R13.1, R2.1, R9.1, TP2.TP, TVS1.1, U1.14, U2.2, X1.1; no longer C1.1, C5.1, C6.2, C7.2, CN1.1, JP2.3, R1.1, R4.1, TVS2.1, U1.2, U2.14, U4.1
- net ICSPCLK: now also JP1.5, U1.12; no longer JP2.5, U2.12
- net ICSPDAT: now also JP1.4, U1.13; no longer JP2.4, U2.13
- net N$1: now also R5.2, U2.5; no longer R1.2, U1.5
- net N$2: now also R7.2, U2.1; no longer R2.2, U1.1
- net N$3: now also LED2.C, R7.1; no longer LED1.C, R2.1
- net N$4: now also R10.2, U1.8; no longer R9.2, U2.8
- net N$8: now also LED1.A, LED3.A, R6.2; no longer TR1.3
- net RESET: now also C1.1, JP1.1, R1.1, U1.4; no longer C7.1, JP2.1, R10.1, U2.4
- net RX: now also R3.2; no longer U2.5
- net SERVO_ON: now also R14.1, U1.9; no longer R6.1, U2.9
- net SERVO_PWM: now also R10.1, X1.3; no longer R9.1
- net TX: now also R4.2; no longer U2.6
- net VBAT: now also CN1.1, D3.A, R14.2, R8.2, U2.3; no longer CN1.2, D4.A, R3.2, R6.2, U1.3
- net VIN: now also D2.C, D3.C; no longer D1.C, D4.C

Commit message: gerber done
Parts:
- moved X1 43.3 mm to (16.6, -8.89), turned to 270 degrees
- moved U3 40.0 mm to (26.1, -2.54)
- moved R6 39.9 mm to (42.6, -5.71), turned to 270 degrees
- moved JP1 38.0 mm to (47.6, -5.08), turned to 90 degrees
- moved R4 36.2 mm to (41.3, -5.71), turned to 270 degrees
- moved C1 35.8 mm to (37.5, -5.08), turned to 0 degrees
- moved R3 35.5 mm to (40.0, -5.71), turned to 270 degrees
- moved TR1 35.5 mm to (19.8, -8.89), turned to 90 degrees
- moved R1 35.1 mm to (34.9, -5.08), turned to 180 degrees
- moved C4 34.7 mm to (29.5, -2.54)
- moved D2 34.7 mm to (25.4, 3.81)
- moved LED1 33.5 mm to (31.3, -8.26), turned to 270 degrees
- moved LED3 33.3 mm to (31.3, -10.2), turned to 0 degrees
- moved D3 32.9 mm to (25.4, 1.91)
- moved C3 32.1 mm to (22.2, -2.54)
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Routing:
- net SERVO_ON: track 0.00 -> 46.8 mm, vias 0 -> 6
- net VBAT: track 0.00 -> 42.8 mm, vias 0 -> 2
- net SERVO_PWM: track 0.00 -> 41.0 mm, vias 0 -> 4
- net +5V: track 0.00 -> 33.9 mm
- net +3.3V: track 0.00 -> 27.5 mm
- net DGND: track 0.00 -> 26.7 mm, vias 0 -> 10
- net N$15: track 0.00 -> 26.2 mm, vias 0 -> 2
- net N$16: track 0.00 -> 26.1 mm, vias 0 -> 2
- net RESET: track 0.00 -> 21.4 mm
- net N$8: track 0.00 -> 18.5 mm
- net VIN: track 0.00 -> 15.1 mm
- net ICSPCLK: track 0.00 -> 14.5 mm
- net ICSPDAT: track 0.00 -> 14.2 mm
- net BAT_ADC: track 0.00 -> 6.17 mm
- net N$2: track 0.00 -> 4.98 mm
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- added copper zone on layer 16, net DGND
Other:
- board size 160 x 100 mm -> 94 x 34.2 mm
- board text added: "2016 Oct"
- board text added: "Hojun Song"
- board text added: "Keep the Water Clean"
- board text added: "ROBOT FISH"

Commit message: value changed
Parts:
- R10, R3, R4: value (none) -> 4.7k
- R2: value 100k -> 1M
Changed lines of the file:
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@@
 <element name="D2" library="microbuilder" package="SOD-123" value="MBR120" x="25.415" y="3.81" rot="R180"/>
 <element name="U1" library="water" package="SO-14" value="16F1575" x="38.75" y="0"/>
-<element name="R2" library="water" package="R0603(1608)" value="100k" x="12.715" y="0" rot="R90"/>
+<element name="R2" library="water" package="R0603(1608)" value="1M" x="12.715" y="0" rot="R90"/>
 <element name="TR1" library="water" package="SOT23" value="SSM3J338R" x="19.795" y="-8.89" rot="R90"/>
 <element name="R14" library="water" package="R0603(1608)" value="100k" x="22.97" y="-8.89" rot="R90"/>
 <element name="C2" library="water" package="C0603(1608)" value="0.1uF" x="33.035" y="0" rot="R90"/>
-<element name="R10" library="water" package="R0603(1608)" value="" x="42.53" y="5.715" rot="R270"/>
+<element name="R10" library="water" package="R0603(1608)" value="4.7k" x="42.53" y="5.715" rot="R270"/>
 <element name="R1" library="water" package="R0603(1608)" value="100k" x="34.94" y="-5.08" rot="R180"/>
 <element name="C1" library="water" package="C0603(1608)" value="0.1uF" x="37.48" y="-5.08"/>
 <element name="D1" library="microbuilder" package="SOD-123" value="MBR120" x="13.985" y="3.175" rot="R180"/>
-<element name="R3" library="water" package="R0603(1608)" value="" x="40.02" y="-5.715" rot="R270"/>
-<element name="R4" library="water" package="R0603(1608)" value="" x="41.29" y="-5.715" rot="R270"/>
+<element name="R3" library="water" package="R0603(1608)" value="4.7k" x="40.02" y="-5.715" rot="R270"/>
+<element name="R4" library="water" package="R0603(1608)" value="4.7k" x="41.29" y="-5.715" rot="R270"/>
 <element name="R6" library="water" package="R0603(1608)" value="1k" x="42.56" y="-5.715" rot="R270"/>
 <element name="LED1" library="berry" package="LED-0603" value="" x="31.2725" y="-8.255" rot="R270"/>
